File: HW/star/star.sch (KiCad schematic (older format))
At the start: 10 parts

Commit message: added gitignor and ref desg
Parts:
- added D5: LED, symbol Device:LED
- added R5: 100R, symbol Device:R
- gave numbers to parts that had none: 10
Connections:
- net labels added: NC
- wire segments 24 -> 30
Changed lines of the file:
@@
 $EndDescr
 $Comp
-L Device:R R?
+L Device:R R1
 U 1 1 5BA87A46
 P 3830 1490
-F 0 "R?" V 3623 1490 50  0000 C CNN
+F 0 "R1" V 3623 1490 50  0000 C CNN
 F 1 "100R" V 3714 1490 50  0000 C CNN
 F 2 "" V 3760 1490 50  0001 C CNN
@@
 $EndComp
 $Comp
-L Device:LED D?
+L Device:LED D1
 U 1 1 5BA87B0E
 P 4260 1490
-F 0 "D?" H 4260 1290 50  0000 C CNN
+F 0 "D1" H 4260 1290 50  0000 C CNN
 F 1 "LED" H 4260 1380 50  0000 C CNN
 F 2 "" H 4260 1490 50  0001 C CNN
@@
 $EndComp
 $Comp
-L MCU_Microchip_ATtiny:ATtiny85V-10SU U?
+L MCU_Microchip_ATtiny:ATtiny85V-10SU U1
 U 1 1 5BA87F89
 P 1910 1900
-F 0 "U?" H 1380 1946 50  0000 R CNN
+F 0 "U1" H 1380 1946 50  0000 R CNN
 F 1 "ATtiny85V-10SU" H 1380 1855 50  0000 R CNN
 F 2 "Package_SO:SOIJ-8_5.3x5.3mm_P1.27mm" H 1910 1900 50  0001 C CIN
@@
 $EndComp
 $Comp
-L Device:Battery_Cell BT?
+L Device:Battery_Cell BT1
 U 1 1 5BA8809B
-P 5180 1990
-F 0 "BT?" H 5298 2086 50  0000 L CNN
-F 1 "Battery_Cell" H 5298 1995 50  0000 L CNN
-F 2 "" V 5180 2050 50  0001 C CNN
-F 3 "~" V 5180 2050 50  0001 C CNN
-	1    5180 1990
-	1    0    0    -1
-$EndComp
-Wire Wire Line
-	5180 1790 5180 1620
-Text Label 5180 1620 0    50   ~ 0
+P 4990 2010
+F 0 "BT1" H 5108 2106 50  0000 L CNN
+F 1 "Battery_Cell" H 5108 2015 50  0000 L CNN
+F 2 "" V 4990 2070 50  0001 C CNN
+F 3 "~" V 4990 2070 50  0001 C CNN
+	1    4990 2010
+	1    0    0    -1
+$EndComp
+Wire Wire Line
+	4990 1810 4990 1640
+Text Label 4990 1640 0    50   ~ 0
 VCC
 Wire Wire Line
@@
 	1910 2670 1910 2500
 $Comp
-L power:GND #PWR?
+L power:GND #PWR01
 U 1 1 5BA883A2
 P 1910 2670
-F 0 "#PWR?" H 1910 2420 50  0001 C CNN
+F 0 "#PWR01" H 1910 2420 50  0001 C CNN
 F 1 "GND" H 1915 2497 50  0000 C CNN
 F 2 "" H 1910 2670 50  0001 C CNN
@@
 $EndComp
 Wire Wire Line
-	5180 2260 5180 2090
-$Comp
-L power:GND #PWR?
+	4990 2280 4990 2110
+$Comp
+L power:GND #PWR03
 U 1 1 5BA883E5
-P 5180 2260
-F 0 "#PWR?" H 5180 2010 50  0001 C CNN
-F 1 "GND" H 5185 2087 50  0000 C CNN
-F 2 "" H 5180 2260 50  0001 C CNN
-F 3 "" H 5180 2260 50  0001 C CNN
-	1    5180 2260
-	1    0    0    -1
-$EndComp
-$Comp
-L Device:R R?
+P 4990 2280
+F 0 "#PWR03" H 4990 2030 50  0001 C CNN
+F 1 "GND" H 4995 2107 50  0000 C CNN
+F 2 "" H 4990 2280 50  0001 C CNN
+F 3 "" H 4990 2280 50  0001 C CNN
+	1    4990 2280
+	1    0    0    -1
+$EndComp
+$Comp
+L Device:R R2
 U 1 1 5BA890DC
 P 3830 1810
-F 0 "R?" V 3623 1810 50  0000 C CNN
+F 0 "R2" V 3623 1810 50  0000 C CNN
 F 1 "100R" V 3714 1810 50  0000 C CNN
 F 2 "" V 3760 1810 50  0001 C CNN
@@
 $EndComp
 $Comp
-L Device:LED D?
+L Device:LED D2
 U 1 1 5BA890E2
 P 4240 1810
-F 0 "D?" H 4240 1610 50  0000 C CNN
+F 0 "D2" H 4240 1610 50  0000 C CNN
 F 1 "LED" H 4240 1700 50  0000 C CNN
 F 2 "" H 4240 1810 50  0001 C CNN
@@
 $EndComp
 $Comp
-L Device:R R?
+L Device:R R3
 U 1 1 5BA8921B
 P 3830 2130
-F 0 "R?" V 3623 2130 50  0000 C CNN
+F 0 "R3" V 3623 2130 50  0000 C CNN
 F 1 "100R" V 3714 2130 50  0000 C CNN
 F 2 "" V 3760 2130 50  0001 C CNN
@@
 $EndComp
 $Comp
-L Device:LED D?
+L Device:LED D3
 U 1 1 5BA89221
 P 4230 2130
-F 0 "D?" H 4230 1930 50  0000 C CNN
+F 0 "D3" H 4230 1930 50  0000 C CNN
 F 1 "LED" H 4230 2020 50  0000 C CNN
 F 2 "" H 4230 2130 50  0001 C CNN
@@
 	3980 2130 4080 2130
 $Comp
-L Device:R R?
+L Device:R R4
 U 1 1 5BA89228
 P 3830 2450
-F 0 "R?" V 3623 2450 50  0000 C CNN
+F 0 "R4" V 3623 2450 50  0000 C CNN
 F 1 "100R" V 3714 2450 50  0000 C CNN
 F 2 "" V 3760 2450 50  0001 C CNN
@@
 $EndComp
 $Comp
-L Device:LED D?
+L Device:LED D4
 U 1 1 5BA8922E
 P 4210 2450
-F 0 "D?" H 4210 2250 50  0000 C CNN
+F 0 "D4" H 4210 2250 50  0000 C CNN
 F 1 "LED" H 4210 2340 50  0000 C CNN
 F 2 "" H 4210 2450 50  0001 C CNN
@@
 	3450 1810 3680 1810
 Text Label 3450 1810 0    50   ~ 0
-LED1
+LED2
 Wire Wire Line
 	3450 2450 3680 2450
 Text Label 3450 2450 0    50   ~ 0
-LED1
+LED4
 Wire Wire Line
 	3450 2130 3680 2130
 Text Label 3450 2130 0    50   ~ 0
-LED1
+LED3
+Wire Wire Line
+	2510 2100 2740 2100
+Text Label 2740 2100 2    50   ~ 0
+NC
+$Comp
+L Device:R R5
+U 1 1 5BA8CB03
+P 3830 2770
+F 0 "R5" V 3623 2770 50  0000 C CNN
+F 1 "100R" V 3714 2770 50  0000 C CNN
+F 2 "" V 3760 2770 50  0001 C CNN
+F 3 "~" H 3830 2770 50  0001 C CNN
+	1    3830 2770
+	0    1    1    0
+$EndComp
+$Comp
+L Device:LED D5
+U 1 1 5BA8CB09
+P 4210 2770
+F 0 "D5" H 4210 2570 50  0000 C CNN
+F 1 "LED" H 4210 2660 50  0000 C CNN
+F 2 "" H 4210 2770 50  0001 C CNN
+F 3 "~" H 4210 2770 50  0001 C CNN
+	1    4210 2770
+	-1   0    0    1
+$EndComp
+Wire Wire Line
+	4520 2770 4360 2770
+Wire Wire Line
+	4060 2770 3980 2770
+Wire Wire Line
+	3450 2770 3680 2770
+Text Label 3450 2770 0    50   ~ 0
+LED5
+Connection ~ 4520 2450
+Wire Wire Line
+	4520 2770 4520 2450
+Wire Wire Line
+	4520 2940 4520 2770
+$Comp
+L power:GND #PWR02
+U 1 1 5BA8E813
+P 4520 2940
+F 0 "#PWR02" H 4520 2690 50  0001 C CNN
+F 1 "GND" H 4525 2767 50  0000 C CNN
+F 2 "" H 4520 2940 50  0001 C CNN
+F 3 "" H 4520 2940 50  0001 C CNN
+	1    4520 2940
+	1    0    0    -1
+$EndComp
+Connection ~ 4520 2770
 $EndSCHEMATC
