File: HW/star.sch (KiCad schematic (older format))
At the start: 12 parts

Commit message: moved directory, added net
Parts:
- D1, D2, D3, D4, D5: renamed from D?; footprint (none) -> LED_THT:LED_D3.0mm
- R1: renamed from R?; footprint (none) -> Resistor_THT:R_Axial_DIN0207_L6.3mm_D2.5mm_P7.62mm_Horizontal
- R2, R5: renamed from R?; footprint (none) -> Resistor_THT:R_Axial_DIN0207_L6.3mm_D2.5mm_P10.16mm_Horizontal
- R3: renamed from R?; footprint (none) -> Resistor_THT:R_Axial_DIN0207_L6.3mm_D2.5mm_P15.24mm_Horizontal
- R4: renamed from R?; footprint (none) -> Resistor_THT:R_Axial_DIN0207_L6.3mm_D2.5mm_P2.54mm_Vertical
- gave numbers to parts that had none: 2
Changed lines of the file:
@@
 $EndDescr
 $Comp
-L Device:R R?
+L Device:R R1
 U 1 1 5BA87A46
 P 3830 1490
-F 0 "R?" V 3623 1490 50  0000 C CNN
+F 0 "R1" V 3623 1490 50  0000 C CNN
 F 1 "100R" V 3714 1490 50  0000 C CNN
-F 2 "" V 3760 1490 50  0001 C CNN
+F 2 "Resistor_THT:R_Axial_DIN0207_L6.3mm_D2.5mm_P7.62mm_Horizontal" V 3760 1490 50  0001 C CNN
 F 3 "~" H 3830 1490 50  0001 C CNN
 	1    3830 1490
@@
 $EndComp
 $Comp
-L Device:LED D?
+L Device:LED D1
 U 1 1 5BA87B0E
 P 4260 1490
-F 0 "D?" H 4260 1290 50  0000 C CNN
+F 0 "D1" H 4260 1290 50  0000 C CNN
 F 1 "LED" H 4260 1380 50  0000 C CNN
-F 2 "" H 4260 1490 50  0001 C CNN
+F 2 "LED_THT:LED_D3.0mm" H 4260 1490 50  0001 C CNN
 F 3 "~" H 4260 1490 50  0001 C CNN
 	1    4260 1490
@@
 $EndComp
 $Comp
-L MCU_Microchip_ATtiny:ATtiny85V-10SU U?
+L MCU_Microchip_ATtiny:ATtiny85V-10SU U1
 U 1 1 5BA87F89
 P 1910 1900
-F 0 "U?" H 1380 1946 50  0000 R CNN
+F 0 "U1" H 1380 1946 50  0000 R CNN
 F 1 "ATtiny85V-10SU" H 1380 1855 50  0000 R CNN
 F 2 "Package_SO:SOIJ-8_5.3x5.3mm_P1.27mm" H 1910 1900 50  0001 C CIN
@@
 $EndComp
 $Comp
-L Device:Battery_Cell BT?
+L Device:Battery_Cell BT1
 U 1 1 5BA8809B
 P 4990 2010
-F 0 "BT?" H 5108 2106 50  0000 L CNN
+F 0 "BT1" H 5108 2106 50  0000 L CNN
 F 1 "Battery_Cell" H 5108 2015 50  0000 L CNN
 F 2 "" V 4990 2070 50  0001 C CNN
@@
 	1910 2670 1910 2500
 $Comp
-L power:GND #PWR?
+L power:GND #PWR01
 U 1 1 5BA883A2
 P 1910 2670
-F 0 "#PWR?" H 1910 2420 50  0001 C CNN
+F 0 "#PWR01" H 1910 2420 50  0001 C CNN
 F 1 "GND" H 1915 2497 50  0000 C CNN
 F 2 "" H 1910 2670 50  0001 C CNN
@@
 	4990 2280 4990 2110
 $Comp
-L power:GND #PWR?
+L power:GND #PWR03
 U 1 1 5BA883E5
 P 4990 2280
-F 0 "#PWR?" H 4990 2030 50  0001 C CNN
+F 0 "#PWR03" H 4990 2030 50  0001 C CNN
 F 1 "GND" H 4995 2107 50  0000 C CNN
 F 2 "" H 4990 2280 50  0001 C CNN
@@
 $EndComp
 $Comp
-L Device:R R?
+L Device:R R2
 U 1 1 5BA890DC
 P 3830 1810
-F 0 "R?" V 3623 1810 50  0000 C CNN
+F 0 "R2" V 3623 1810 50  0000 C CNN
 F 1 "100R" V 3714 1810 50  0000 C CNN
-F 2 "" V 3760 1810 50  0001 C CNN
+F 2 "Resistor_THT:R_Axial_DIN0207_L6.3mm_D2.5mm_P10.16mm_Horizontal" V 3760 1810 50  0001 C CNN
 F 3 "~" H 3830 1810 50  0001 C CNN
 	1    3830 1810
@@
 $EndComp
 $Comp
-L Device:LED D?
+L Device:LED D2
 U 1 1 5BA890E2
 P 4240 1810
-F 0 "D?" H 4240 1610 50  0000 C CNN
+F 0 "D2" H 4240 1610 50  0000 C CNN
 F 1 "LED" H 4240 1700 50  0000 C CNN
-F 2 "" H 4240 1810 50  0001 C CNN
+F 2 "LED_THT:LED_D3.0mm" H 4240 1810 50  0001 C CNN
 F 3 "~" H 4240 1810 50  0001 C CNN
 	1    4240 1810
@@
 $EndComp
 $Comp
-L Device:R R?
+L Device:R R3
 U 1 1 5BA8921B
 P 3830 2130
-F 0 "R?" V 3623 2130 50  0000 C CNN
+F 0 "R3" V 3623 2130 50  0000 C CNN
 F 1 "100R" V 3714 2130 50  0000 C CNN
-F 2 "" V 3760 2130 50  0001 C CNN
+F 2 "Resistor_THT:R_Axial_DIN0207_L6.3mm_D2.5mm_P15.24mm_Horizontal" V 3760 2130 50  0001 C CNN
 F 3 "~" H 3830 2130 50  0001 C CNN
 	1    3830 2130
@@
 $EndComp
 $Comp
-L Device:LED D?
+L Device:LED D3
 U 1 1 5BA89221
 P 4230 2130
-F 0 "D?" H 4230 1930 50  0000 C CNN
+F 0 "D3" H 4230 1930 50  0000 C CNN
 F 1 "LED" H 4230 2020 50  0000 C CNN
-F 2 "" H 4230 2130 50  0001 C CNN
+F 2 "LED_THT:LED_D3.0mm" H 4230 2130 50  0001 C CNN
 F 3 "~" H 4230 2130 50  0001 C CNN
 	1    4230 2130
@@
 	3980 2130 4080 2130
 $Comp
-L Device:R R?
+L Device:R R4
 U 1 1 5BA89228
 P 3830 2450
-F 0 "R?" V 3623 2450 50  0000 C CNN
+F 0 "R4" V 3623 2450 50  0000 C CNN
 F 1 "100R" V 3714 2450 50  0000 C CNN
-F 2 "" V 3760 2450 50  0001 C CNN
+F 2 "Resistor_THT:R_Axial_DIN0207_L6.3mm_D2.5mm_P2.54mm_Vertical" V 3760 2450 50  0001 C CNN
 F 3 "~" H 3830 2450 50  0001 C CNN
 	1    3830 2450
@@
 $EndComp
 $Comp
-L Device:LED D?
+L Device:LED D4
 U 1 1 5BA8922E
 P 4210 2450
-F 0 "D?" H 4210 2250 50  0000 C CNN
+F 0 "D4" H 4210 2250 50  0000 C CNN
 F 1 "LED" H 4210 2340 50  0000 C CNN
-F 2 "" H 4210 2450 50  0001 C CNN
+F 2 "LED_THT:LED_D3.0mm" H 4210 2450 50  0001 C CNN
 F 3 "~" H 4210 2450 50  0001 C CNN
 	1    4210 2450
@@
 NC
 $Comp
-L Device:R R?
+L Device:R R5
 U 1 1 5BA8CB03
 P 3830 2770
-F 0 "R?" V 3623 2770 50  0000 C CNN
+F 0 "R5" V 3623 2770 50  0000 C CNN
 F 1 "100R" V 3714 2770 50  0000 C CNN
-F 2 "" V 3760 2770 50  0001 C CNN
+F 2 "Resistor_THT:R_Axial_DIN0207_L6.3mm_D2.5mm_P10.16mm_Horizontal" V 3760 2770 50  0001 C CNN
 F 3 "~" H 3830 2770 50  0001 C CNN
 	1    3830 2770
@@
 $EndComp
 $Comp
-L Device:LED D?
+L Device:LED D5
 U 1 1 5BA8CB09
 P 4210 2770
-F 0 "D?" H 4210 2570 50  0000 C CNN
+F 0 "D5" H 4210 2570 50  0000 C CNN
 F 1 "LED" H 4210 2660 50  0000 C CNN
-F 2 "" H 4210 2770 50  0001 C CNN
+F 2 "LED_THT:LED_D3.0mm" H 4210 2770 50  0001 C CNN
 F 3 "~" H 4210 2770 50  0001 C CNN
 	1    4210 2770
@@
 	4520 2940 4520 2770
 $Comp
-L power:GND #PWR?
+L power:GND #PWR02
 U 1 1 5BA8E813
 P 4520 2940
-F 0 "#PWR?" H 4520 2690 50  0001 C CNN
+F 0 "#PWR02" H 4520 2690 50  0001 C CNN
 F 1 "GND" H 4525 2767 50  0000 C CNN
 F 2 "" H 4520 2940 50  0001 C CNN

Commit message: done with layout
Parts:
- BT1: footprint (none) -> star:CR2030_Retainer
- R2, R5: footprint Resistor_THT:R_Axial_DIN0207_L6.3mm_D2.5mm_P10.16mm_Horizontal -> Resistor_THT:R_Axial_DIN0207_L6.3mm_D2.5mm_P7.62mm_Horizontal
- R3: footprint Resistor_THT:R_Axial_DIN0207_L6.3mm_D2.5mm_P15.24mm_Horizontal -> Resistor_THT:R_Axial_DIN0207_L6.3mm_D2.5mm_P7.62mm_Horizontal
- R4: footprint Resistor_THT:R_Axial_DIN0207_L6.3mm_D2.5mm_P2.54mm_Vertical -> Resistor_THT:R_Axial_DIN0207_L6.3mm_D2.5mm_P7.62mm_Horizontal
Changed lines of the file:
@@
 EESchema Schematic File Version 4
+LIBS:star-cache
 EELAYER 26 0
 EELAYER END
@@
 F 0 "BT1" H 5108 2106 50  0000 L CNN
 F 1 "Battery_Cell" H 5108 2015 50  0000 L CNN
-F 2 "" V 4990 2070 50  0001 C CNN
+F 2 "star:CR2030_Retainer" V 4990 2070 50  0001 C CNN
 F 3 "~" V 4990 2070 50  0001 C CNN
 	1    4990 2010
@@
 F 0 "R2" V 3623 1810 50  0000 C CNN
 F 1 "100R" V 3714 1810 50  0000 C CNN
-F 2 "Resistor_THT:R_Axial_DIN0207_L6.3mm_D2.5mm_P10.16mm_Horizontal" V 3760 1810 50  0001 C CNN
+F 2 "Resistor_THT:R_Axial_DIN0207_L6.3mm_D2.5mm_P7.62mm_Horizontal" V 3760 1810 50  0001 C CNN
 F 3 "~" H 3830 1810 50  0001 C CNN
 	1    3830 1810
@@
 F 0 "R3" V 3623 2130 50  0000 C CNN
 F 1 "100R" V 3714 2130 50  0000 C CNN
-F 2 "Resistor_THT:R_Axial_DIN0207_L6.3mm_D2.5mm_P15.24mm_Horizontal" V 3760 2130 50  0001 C CNN
+F 2 "Resistor_THT:R_Axial_DIN0207_L6.3mm_D2.5mm_P7.62mm_Horizontal" V 3760 2130 50  0001 C CNN
 F 3 "~" H 3830 2130 50  0001 C CNN
 	1    3830 2130
@@
 F 0 "R4" V 3623 2450 50  0000 C CNN
 F 1 "100R" V 3714 2450 50  0000 C CNN
-F 2 "Resistor_THT:R_Axial_DIN0207_L6.3mm_D2.5mm_P2.54mm_Vertical" V 3760 2450 50  0001 C CNN
+F 2 "Resistor_THT:R_Axial_DIN0207_L6.3mm_D2.5mm_P7.62mm_Horizontal" V 3760 2450 50  0001 C CNN
 F 3 "~" H 3830 2450 50  0001 C CNN
 	1    3830 2450
@@
 F 0 "R5" V 3623 2770 50  0000 C CNN
 F 1 "100R" V 3714 2770 50  0000 C CNN
-F 2 "Resistor_THT:R_Axial_DIN0207_L6.3mm_D2.5mm_P10.16mm_Horizontal" V 3760 2770 50  0001 C CNN
+F 2 "Resistor_THT:R_Axial_DIN0207_L6.3mm_D2.5mm_P7.62mm_Horizontal" V 3760 2770 50  0001 C CNN
 F 3 "~" H 3830 2770 50  0001 C CNN
 	1    3830 2770
