File: HW/star.kicad_pcb (KiCad board)
At the start: 2 copper layers, 50.4 x 48 mm, 21 parts, among them U1 ATtiny85V-10SU

Commit message: idk stuff changed
Parts:
- removed the G*** at (118.3, 79.2) (x4)
- added G*** (x4): LOGO, LOGO, F.Cu at (118.3, 79.2)
- moved R3 1.94 mm to (127.1, 95.5), turned to 147 degrees
- moved R4 1.18 mm to (109.5, 95.5)
Routing:
- net GND: track 1.93 -> 46.1 mm, vias 0 -> 3
- net /VCC: track 0.00 -> 28.0 mm, vias 0 -> 1
- net /LED3: track 9.30 -> 12.3 mm
- net Net-(D3-Pad2): track 2.94 -> 2.15 mm
- net /LED4: track 13.0 -> 12.4 mm
